File: finalhe.kicad_sch (KiCad schematic)
At the start: 20 parts, among them P1 USB_C_Plug_USB2.0, SW1 SW_Push, SW2 SW_SPDT, U1 STM32F070F6Px, U5 TLV1117-33, Y1 8MHz 18pF

Commit message: fdsfkjsdh
Parts:
- added C58: 1uF, symbol Device:C
- added R53: 1k, symbol Device:R
- C3: value 1uF -> 100nF
Connections:
- net +3.3V: now also SW2.3 (C), C58.2; no longer FB1.1, SW2.1 (A)
- net GND: now also C3.2, C4.2, C56.2, C57.2, SW2.1 (A), Y1.2, Y1.4; no longer SW2.3 (C)
- net OSC_OUT: now also R53.2; no longer C57.1, Y1.3
- new net: C57.1, R53.1, Y1.3
- new net: C58.1, FB1.1
- no-connect marks 1 -> 2
Other:
- moved on the sheet: C56, C57
