File: Multiplexer.kicad_sch (KiCad schematic)
At the start: 1 part, among them U2 CD74HC4067SM

Commit message: fdsfkjsdh
Parts:
- added C59: 100nF, symbol Device:C
Connections:
- net +3.3V: now also C59.2
- net GND: now also C59.1
Changed lines of the file:
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@@
 (kicad_sch (version 20230121) (generator eeschema)
   (paper "A4")
+  (junction (at 88.9 73.66) (diameter 0) (color 0 0 0 0)
+  )
   (junction (at 88.9 130.175) (diameter 0) (color 0 0 0 0)
   )
@@
     (stroke (width 0) (type default))
   )
+  (wire (pts (xy 88.9 73.66) (xy 88.9 76.835))
+    (stroke (width 0) (type default))
+  )
   (wire (pts (xy 101.6 92.075) (xy 118.745 92.075))
     (stroke (width 0) (type default))
@@
     (stroke (width 0) (type default))
   )
-  (wire (pts (xy 88.9 76.2) (xy 88.9 76.835))
+  (wire (pts (xy 88.9 71.755) (xy 88.9 73.66))
     (stroke (width 0) (type default))
   )
@@
   )
   (wire (pts (xy 118.745 92.075) (xy 118.745 57.785))
+    (stroke (width 0) (type default))
+  )
+  (wire (pts (xy 80.01 73.66) (xy 81.28 73.66))
     (stroke (width 0) (type default))
   )
@@
     )
   )
-  (symbol (lib_id "power:+3.3V") (at 88.9 76.2 0) (unit 1)
+  (symbol (lib_id "Device:C") (at 85.09 73.66 90) (unit 1)
+    (in_bom yes) (on_board yes) (dnp no)
+    (property "Reference" "C59" (at 85.09 77.47 90)
+      (effects (font (size 1.27 1.27)))
+    )
+    (property "Value" "100nF" (at 85.09 70.485 90)
+      (effects (font (size 1.27 1.27)))
+    )
+    (property "Footprint" "" (at 88.9 72.6948 0)
+      (effects (font (size 1.27 1.27)) hide)
+    )
+    (property "Datasheet" "~" (at 85.09 73.66 0)
+      (effects (font (size 1.27 1.27)) hide)
+    )
+    (pin "2")
+    (pin "1")
+    (instances
+      (project "finalhe"
+        (path "/0c04b3a2-e8e1-4ec6-a192-c07d3f315f4c/4ee3e8cf-5365-4e52-b7b7-187536c01e8d"
+          (reference "C59") (unit 1)
+        )
+        (path "/0c04b3a2-e8e1-4ec6-a192-c07d3f315f4c/300ee4b1-70ff-4528-bcda-bf08a841fdcb"
+          (reference "C60") (unit 1)
+        )
+        (path "/0c04b3a2-e8e1-4ec6-a192-c07d3f315f4c/7051a185-9438-46b5-913c-99c48ae04508"
+          (reference "C61") (unit 1)
+        )
+      )
+    )
+  )
+  (symbol (lib_id "power:+3.3V") (at 88.9 71.755 0) (unit 1)
     (in_bom yes) (on_board yes) (dnp no) (fields_autoplaced)
-    (property "Reference" "#PWR058" (at 88.9 80.01 0)
-      (effects (font (size 1.27 1.27)) hide)
-    )
-    (property "Value" "+3.3V" (at 88.9 71.755 0)
+    (property "Reference" "#PWR058" (at 88.9 75.565 0)
+      (effects (font (size 1.27 1.27)) hide)
+    )
+    (property "Value" "+3.3V" (at 88.9 67.31 0)
       (effects (font (size 1.27 1.27)))
     )
-    (property "Footprint" "" (at 88.9 76.2 0)
-      (effects (font (size 1.27 1.27)) hide)
-    )
-    (property "Datasheet" "" (at 88.9 76.2 0)
+    (property "Footprint" "" (at 88.9 71.755 0)
+      (effects (font (size 1.27 1.27)) hide)
+    )
+    (property "Datasheet" "" (at 88.9 71.755 0)
       (effects (font (size 1.27 1.27)) hide)
     )
@@
         )
       )
+    )
+  )
+  (symbol (lib_id "power:GND") (at 80.01 73.66 0) (unit 1)
+    (in_bom yes) (on_board yes) (dnp no) (fields_autoplaced)
+    (property "Reference" "#PWR0168" (at 80.01 80.01 0)
+      (effects (font (size 1.27 1.27)) hide)
+    )
+    (property "Value" "GND" (at 80.01 78.74 0)
+      (effects (font (size 1.27 1.27)))
+    )
+    (property "Footprint" "" (at 80.01 73.66 0)
+      (effects (font (size 1.27 1.27)) hide)
+    )
+    (property "Datasheet" "" (at 80.01 73.66 0)
+      (effects (font (size 1.27 1.27)) hide)
+    )
+    (pin "1")
+    (instances
+      (project "finalhe"
+        (path "/0c04b3a2-e8e1-4ec6-a192-c07d3f315f4c/4ee3e8cf-5365-4e52-b7b7-187536c01e8d"
+          (reference "#PWR0168") (unit 1)
+        )
+        (path "/0c04b3a2-e8e1-4ec6-a192-c07d3f315f4c/300ee4b1-70ff-4528-bcda-bf08a841fdcb"
+          (reference "#PWR0169") (unit 1)
+        )
+        (path "/0c04b3a2-e8e1-4ec6-a192-c07d3f315f4c/7051a185-9438-46b5-913c-99c48ae04508"
+          (reference "#PWR0170") (unit 1)
+        )
+      )

Commit message: fdsb
Parts:
- added C63: 1nF, symbol Device:C
- added C65: 100nF, symbol Device:C
- added R55: 100, symbol Device:R
- added U7: TLV9061xDCK, Package_TO_SOT_SMD:SOT-353_SC-70-5, symbol Amplifier_Operational:TLV9061xDCK
Connections:
- net GND: now also C63.2, C65.1, U7.2 (V-)
- net MUX_OUTPUT: now also C63.1, R55.1; no longer U2.1 (COM)
- new net: U2.1 (COM), U7.1 (+)
- new net: R55.2, U7.3 (-), U7.4
- new net VCC: C65.2, U7.5 (V+)
