File: sensor.kicad_sch (KiCad schematic)
At the start: 3 parts

Commit message: fdsfkjsdh
Parts:
- C31: renamed from C8; value 100nF -> 1uF
- R28: renamed from R7; value 10k -> 1k
- renumbered S4 to S25

Commit message: fdsb
Parts:
- renumbered C31 to C8, R28 to R7, S25 to S4
